Commit message: commenting base_footprint, restoring original meshes

File: limo_description/urdf/limo.xacro (robot description, xacro)
@@ -15,7 +15,7 @@
             </visual>
             <collision>
-              <origin xyz="0 ${wheel_length/2} 0" rpy="1.57 0 0" />
+                  <origin xyz="0 0 0" rpy="0 0 0" />
               <geometry>
-                  <cylinder length="${wheel_length}" radius="${wheel_radius}" />
+                  <mesh filename="file://$(find limo_description)/meshes/limo_optimal_wheels.dae" />
               </geometry>
             </collision>

File: limo_description/urdf/limo_four_diff.xacro (robot description, xacro)
@@ -17,10 +17,10 @@
 	    <xacro:property name="wheel_length" value="0.045" />
 	    <xacro:property name="wheel_radius" value="0.045" />
-	  <link name="limo${robot_id}/base_footprint"/>
-	  <joint name="limo${robot_id}/base_joint" type="fixed">
+	  <!--link name="limo${robot_id}/base_footprint"/-->
+	  <!--joint name="limo${robot_id}/base_joint" type="fixed">
 	    <parent link="limo${robot_id}/base_footprint"/>
 	    <child link="limo${robot_id}/base_link"/>
 	    <origin xyz="0.0 0.0 0.15" rpy="0 0 0"/>
-	  </joint>
+	  </joint-->
 	    <!-- Base link -->
 	    <link name="limo${robot_id}/base_link">
@@ -33,7 +33,7 @@
 		<collision>
 		    <!--origin xyz="0 0 -0.15" rpy="0 0 1.57" /-->
-		    <origin xyz="0 0 0" rpy="0 0 0" />
+		    <origin xyz="0 0 -0.15" rpy="0 0 1.57" />
 		  <geometry>
-		      <box size="${base_x_size} ${base_y_size} ${base_z_size}"/>
+		      <mesh filename="file://$(find limo_description)/meshes/limo_optimal.dae" scale="1 1 1"/>
 		  </geometry>
 		</collision>

Commit message: hack to reduce friction and improve tracking: 1) set back wheelsas passive 2) reduce friction on back wheels 3) replace cylinders in place of wheel CAD

File: limo_description/urdf/limo.xacro (robot description, xacro)
@@ -15,9 +15,15 @@
             </visual>
             <collision>
+              <origin xyz="0 ${wheel_length/2} 0" rpy="1.57 0 0" />
+              <geometry>
+                  <cylinder length="${wheel_length}" radius="${wheel_radius}" />
+              </geometry>
+            </collision>
+            <!--collision>
                   <origin xyz="0 0 0" rpy="0 0 0" />
               <geometry>
                   <mesh filename="file://$(find limo_description)/meshes/limo_optimal_wheels.dae" />
               </geometry>
-            </collision>
+            </collision-->
         </link>
         <joint name="${wheel_prefix}_wheel" type="continuous">

File: limo_description/urdf/limo_four_diff.xacro (robot description, xacro)
@@ -83,5 +83,5 @@
         <mu1>1.</mu1>
         <mu2>1.</mu2>
-        <kp>10000000.0</kp>
+        <kp>1000000.0</kp>
         <kd>1.0</kd>
         <maxVel>1.0</maxVel>
@@ -91,5 +91,5 @@
         <mu1>1.</mu1>
         <mu2>1.</mu2>
-        <kp>10000000.0</kp>
+        <kp>1000000.0</kp>
         <kd>1.0</kd>
         <maxVel>1.0</maxVel>
@@ -97,7 +97,7 @@
     </gazebo>
     <gazebo reference="limo${robot_id}/rear_left_wheel_link">
-        <mu1>1.</mu1>
-        <mu2>1.</mu2>
-        <kp>10000000.0</kp>
+        <mu1>0.5</mu1> <!--DIRTY TRICK TO SOLVE ISSUE OF BAD TRACKING DUE TO FRICTION-->
+        <mu2>0.5</mu2>
+        <kp>1000000.0</kp>
         <kd>1.0</kd>
         <maxVel>1.0</maxVel>
@@ -105,7 +105,7 @@
     </gazebo>
     <gazebo reference="limo${robot_id}/rear_right_wheel_link">
-        <mu1>1.</mu1>
-        <mu2>1.</mu2>
-        <kp>10000000.0</kp>
+        <mu1>0.5</mu1> <!--DIRTY TRICK TO SOLVE ISSUE OF BAD TRACKING DUE TO FRICTION-->
+        <mu2>0.5</mu2>
+        <kp>1000000.0</kp>
         <kd>1.0</kd>
         <maxVel>1.0</maxVel>
@@ -117,14 +117,14 @@
 		    <!-- Put all ROS topics inside this namespace -->
 		    <ros>
-		      <namespace>limo$(arg robot_id)</namespace>
+		      <nameSpace>limo$(arg robot_id)</nameSpace>
 		    </ros>
 		    <updateRate>50</updateRate>
 		    <!-- EXACT joint names from your URDF (underscored) -->
 		    <leftJoint>limo$(arg robot_id)/front_left_wheel</leftJoint>
-		    <leftJoint>limo$(arg robot_id)/rear_left_wheel</leftJoint>
 		    <rightJoint>limo$(arg robot_id)/front_right_wheel</rightJoint>
-		    <rightJoint>limo$(arg robot_id)/rear_right_wheel</rightJoint>
+ 		    <!--leftJoint>limo$(arg robot_id)/rear_left_wheel</leftJoint--> <!--DIRTY TRICK TO SOLVE ISSUE OF BAD TRACKING DUE TO FRICTION-->
+ 		    <!--rightJoint>limo$(arg robot_id)/rear_right_wheel</rightJoint--> <!--DIRTY TRICK TO SOLVE ISSUE OF BAD TRACKING DUE TO FRICTION-->
 		    <wheelSeparation>0.164</wheelSeparation>
-		    <wheelDiameter>0.08</wheelDiameter>
+		    <wheelDiameter>0.09</wheelDiameter>
 		    <!-- Topics are relative to the namespace above -->
 		    <commandTopic>cmd_vel</commandTopic>

Commit message: added labirinth, fixed laser sensor

File: limo_description/urdf/limo.xacro (robot description, xacro)
@@ -20,11 +20,5 @@
               </geometry>
             </collision>
-            <!--collision>
-                  <origin xyz="0 0 0" rpy="0 0 0" />
-              <geometry>
-                  <mesh filename="file://$(find limo_description)/meshes/limo_optimal_wheels.dae" />
-              </geometry>
-            </collision-->
-        </link>
+           </link>
         <joint name="${wheel_prefix}_wheel" type="continuous">
             <parent link="${parent_prefix}"/>

File: limo_description/urdf/limo_four_diff.xacro (robot description, xacro)
@@ -2,7 +2,8 @@
 <robot name="limo" xmlns:xacro="http://ros.org/wiki/xacro">
     <xacro:arg name="robot_id" default="" />
-	     <xacro:macro name="limo" params='robot_id'>
+    <xacro:arg name="sensors" default="true" />
+     <xacro:macro name="limo_robot" params='robot_id'>
 	    <!-- defines limo wheel, laser, depth camera, imu macros-->
-	    <xacro:include filename="$(find limo_description)/urdf/limo.xacro" />
+    	    <xacro:include filename="$(find limo_description)/urdf/limo.xacro" />
 	    <!-- Variables -->
 	    <xacro:property name="M_PI" value="3.14159"/>
@@ -28,5 +29,5 @@
 		    <origin xyz="0 0 -0.15" rpy="0 0 1.57" />
 		    <geometry>
-		        <mesh filename="file://$(find limo_description)/meshes/limo_optimal.dae" scale="1 1 1"/>
+		        <mesh filename="file://$(find limo_description)/meshes/limo_base.dae" scale="1 1 1"/>
 		    </geometry>
 		</visual>
@@ -35,5 +36,5 @@
 		    <origin xyz="0 0 -0.15" rpy="0 0 1.57" />
 		  <geometry>
-		      <mesh filename="file://$(find limo_description)/meshes/limo_optimal.dae" scale="1 1 1"/>
+		      <mesh filename="file://$(find limo_description)/meshes/limo_base.dae" scale="1 1 1"/>
 		  </geometry>
 		</collision>
@@ -162,10 +163,15 @@
 		   <plugin name="joint_state_pub" filename="libgazebo_ros_joint_state_publisher.so">
 		    <ros><namespace>limo$(arg robot_id)</namespace></ros>
-		    <updateRate>50</updateRate>
+		    <updateRate>100</updateRate>
                      <alwaysOn>true</alwaysOn>
 	              <jointName>limo$(arg robot_id)/front_left_wheel, limo$(arg robot_id)/rear_left_wheel,limo$(arg robot_id)/front_right_wheel,limo$(arg robot_id)/rear_right_wheel</jointName>
 		  </plugin>
 	</gazebo>
+    <xacro:if value="$(arg sensors)">
+            <xacro:include filename="$(find limo_description)/urdf/limo_sensors.gazebo" />
+      	    <xacro:limo_sensors robot_id="$(arg robot_id)"/>
+      </xacro:if>
     </xacro:macro>
-    <xacro:limo robot_id="$(arg robot_id)" />
+    <!-- instantiate the actual robot -->
+    <xacro:limo_robot robot_id="$(arg robot_id)" />
 </robot>
