Commit message: one limu works with ros control

File: limo_description/urdf/limo_four_diff.xacro (robot description, xacro)
@@ -3,246 +3,85 @@
     <xacro:arg name="robot_id" default="" />
     <xacro:macro name="limo" params='robot_id'>
-    <xacro:include filename="$(find limo_description)/urdf/limo.xacro" />
-    <xacro:include filename="$(find limo_description)/urdf/limo_four_diff.gazebo" />
-    <!-- Variables -->
-    <xacro:property name="M_PI" value="3.14159"/>
-    <!-- Vehicle Geometries -->
-    <xacro:property name="base_x_size" value="0.13" />
-    <xacro:property name="base_y_size" value="0.12" />
-    <xacro:property name="base_z_size" value="0.1" />
-    <xacro:property name="wheelbase" value="0.2"/>
-    <xacro:property name="track" value="0.13"/>
-    <xacro:property name="wheel_vertical_offset" value="-0.10" />
-    <xacro:property name="base_mass" value="2.1557"/>
-    <xacro:property name="wheel_length" value="0.045" />
-    <xacro:property name="wheel_radius" value="0.045" />
-  <link name="limo${robot_id}/base_footprint"/>
-  <joint name="limo${robot_id}/base_joint" type="fixed">
-    <parent link="limo${robot_id}/base_footprint"/>
-    <child link="limo${robot_id}/base_link"/>
-    <origin xyz="0.0 0.0 0.15" rpy="0 0 0"/>
-  </joint>
-    <!-- Base link -->
-    <link name="limo${robot_id}/base_link">
-        <visual>
-            <origin xyz="0 0 -0.15" rpy="0 0 1.57" />
-            <geometry>
-                <mesh filename="file://$(find limo_description)/meshes/limo_optimal.dae" scale="1 1 1"/>
-            </geometry>
-        </visual>
-        <collision>
-            <!--origin xyz="0 0 -0.15" rpy="0 0 1.57" /-->
-            <origin xyz="0 0 0" rpy="0 0 0" />
-          <geometry>
-              <box size="${base_x_size} ${base_y_size} ${base_z_size}"/>
-          </geometry>
-        </collision>
-    </link>
-    <link name="limo${robot_id}/inertial_link">
-        <inertial>
-            <origin xyz="0.0 0.0 0.0" />
-            <mass value="${base_mass}" />
-            <inertia ixx="0.24" ixy="0" ixz="0"
-                     iyy="0.96" iyz="0"
-                     izz="0.96" />
-        </inertial>
-    </link>
-    <joint name="limo${robot_id}/inertial_joint" type="fixed">
-        <origin xyz="0 0 0" rpy="0 0 0" />
-        <parent link="limo${robot_id}/base_link" />
-        <child link="limo${robot_id}/inertial_link" />
-    </joint>
-    <xacro:limo_laser parent_prefix="limo${robot_id}/base_link" frame_prefix="limo${robot_id}/laser">
-        <origin xyz="0.103 0 -0.034" rpy="0 0 0"/>
-    </xacro:limo_laser>
-    <xacro:limo_depth_camera parent_prefix="limo${robot_id}/base_link" frame_prefix="limo${robot_id}/depth_camera">
-        <origin xyz="0.084 0 0.03" rpy="0 0 0"/>
-    </xacro:limo_depth_camera>
-    <xacro:limo_imu parent_prefix="limo${robot_id}/base_link" frame_prefix="limo${robot_id}/imu">
-        <origin xyz="0.0 0 -0.1" rpy="0 0 0"/>
-    </xacro:limo_imu>
-    <xacro:limo_wheel parent_prefix="limo${robot_id}/base_link" wheel_prefix="limo${robot_id}/front_left" reflect="1">
-        <origin xyz="${wheelbase/2} ${track/2} ${wheel_vertical_offset}" rpy="0 0  0" />
-    </xacro:limo_wheel>
-    <xacro:limo_wheel parent_prefix="limo${robot_id}/base_link" wheel_prefix="limo${robot_id}/front_right" reflect="-1">
-        <origin xyz="${wheelbase/2} ${-track/2} ${wheel_vertical_offset}" rpy="${M_PI} 0 0" />
-    </xacro:limo_wheel>
-    <xacro:limo_wheel parent_prefix="limo${robot_id}/base_link" wheel_prefix="limo${robot_id}/rear_left" reflect="1">
-        <origin xyz="${-wheelbase/2} ${track/2} ${wheel_vertical_offset}" rpy="0 0 0" />
-    </xacro:limo_wheel>
-    <xacro:limo_wheel parent_prefix="limo${robot_id}/base_link" wheel_prefix="limo${robot_id}/rear_right" reflect="-1">
-        <origin xyz="${-wheelbase/2} ${-track/2} ${wheel_vertical_offset}" rpy="${M_PI} 0 0" />
-    </xacro:limo_wheel>
-    <gazebo reference="limo${robot_id}/imu_link">
-    <gravity>true</gravity>
-    <sensor name="twr_imu" type="imu">
-      <always_on>true</always_on>
-      <update_rate>100</update_rate>
-      <visualize>true</visualize>
-      <imu>
-        <orientation>
-          <x>
-            <noise type="gaussian">
-              <mean>0.0</mean>
-              <stddev>2e-3</stddev>
-            </noise>
-          </x>
-          <y>
-            <noise type="gaussian">
-              <mean>0.0</mean>
-              <stddev>2e-3</stddev>
-            </noise>
-          </y>
-          <z>
-            <noise type="gaussian">
-              <mean>0.0</mean>
-              <stddev>2e-3</stddev>
-            </noise>
-          </z>
-        </orientation>
-        <angular_velocity>
-          <x>
-            <noise type="gaussian">
-              <mean>0.0</mean>
-              <stddev>2e-4</stddev>
-            </noise>
-          </x>
-          <y>
-            <noise type="gaussian">
-              <mean>0.0</mean>
-              <stddev>2e-4</stddev>
-            </noise>
-          </y>
-          <z>
-            <noise type="gaussian">
-              <mean>0.0</mean>
-              <stddev>2e-4</stddev>
-            </noise>
-          </z>
-        </angular_velocity>
-        <linear_acceleration>
-          <x>
-            <noise type="gaussian">
-              <mean>0.0</mean>
-              <stddev>1.7e-2</stddev>
-            </noise>
-          </x>
-          <y>
-            <noise type="gaussian">
-              <mean>0.0</mean>
-              <stddev>1.7e-2</stddev>
-            </noise>
-          </y>
-          <z>
-            <noise type="gaussian">
-              <mean>0.0</mean>
-              <stddev>1.7e-2</stddev>
-            </noise>
-          </z>
-        </linear_acceleration>
-      </imu>
-      <plugin name="two_wheeled_robot_imu" filename="libgazebo_ros_imu_sensor.so">
-        <initial_orientation_as_reference>false</initial_orientation_as_reference>
-        <frame_name>limo${robot_id}/imu_link</frame_name>
-        <ros>
-          <remapping>~/out:=data</remapping>
-        </ros>
-      </plugin>
-    </sensor>
-</gazebo>
-<gazebo reference="limo${robot_id}/laser_link">
-    <sensor name="laser" type="ray">
-      <always_on>true</always_on>
-      <visualize>false</visualize>
-      <update_rate>10</update_rate>
-      <ray>
-        <scan>
-          <horizontal>
-            <samples>120</samples>
-            <resolution>1.000000</resolution>
-            <min_angle>-3.14159</min_angle>
-            <max_angle>3.14159</max_angle>
-          </horizontal>
-        </scan>
-        <range>
-          <min>0.3</min>
-          <max>15.0</max>
-          <resolution>0.015</resolution>
-        </range>
-        <noise>
-          <type>gaussian</type>
-          <mean>0.0</mean>
-          <stddev>0.01</stddev>
-        </noise>
-      </ray>
-      <plugin name="scan" filename="libgazebo_ros_ray_sensor.so">
-        <ros>
-          <remapping>~/out:=scan</remapping>
-        </ros>
-        <output_type>sensor_msgs/LaserScan</output_type>
-        <frame_name>limo${robot_id}/laser_link</frame_name>
-      </plugin>
-    </sensor>
-  </gazebo>
-    <gazebo reference="limo${robot_id}/front_left_wheel">
-        <mu1>100</mu1>
-        <mu2>100</mu2>
-        <kp>10000000.0</kp>
-        <kd>1.0</kd>
-        <minDepth>0.01</minDepth>
-        <fdir1>1 0 0</fdir1>
-        <maxContacts value="64"/>
-    </gazebo>
-    <gazebo reference="limo${robot_id}/front_right_wheel">
-        <mu1>100</mu1>
-        <mu2>100</mu2>
-        <kp>10000000.0</kp>
-        <kd>1.0</kd>
-        <minDepth>0.01</minDepth>
-        <fdir1>1 0 0</fdir1>
-        <maxContacts value="64"/>
-    </gazebo>
-    <gazebo reference="limo${robot_id}/rear_left_wheel">
-        <mu1>100</mu1>
-        <mu2>100</mu2>
-        <kp>10000000.0</kp>
-        <kd>1.0</kd>
-        <minDepth>0.01</minDepth>
-        <fdir1>1 0 0</fdir1>
-        <maxContacts value="64"/>
-    </gazebo>
-    <gazebo reference="limo${robot_id}/rear_right_wheel">
-        <mu1>100</mu1>
-        <mu2>100</mu2>
-        <kp>10000000.0</kp>
-        <kd>1.0</kd>
-        <minDepth>0.01</minDepth>
-        <fdir1>1 0 0</fdir1>
-        <maxContacts value="64"/>
-    </gazebo>
-    <gazebo>
-        <plugin name="four_diff_controller" filename="libgazebo_ros_diff_drive.so">
-        <update_rate>50</update_rate>
-        <num_wheel_pairs>2</num_wheel_pairs>
-        <left_joint>limo${robot_id}/front_left_wheel</left_joint>
-        <right_joint>limo${robot_id}/front_right_wheel</right_joint>
-        <left_joint>limo${robot_id}/rear_left_wheel</left_joint>
-        <right_joint>limo${robot_id}/rear_right_wheel</right_joint>
-        <wheel_separation>0.172</wheel_separation>
-        <wheel_diameter>0.09</wheel_diameter>
-        <max_wheel_torque>20</max_wheel_torque>
-        <max_wheel_acceleration>1.0</max_wheel_acceleration>
-        <command_topic>limo${robot_id}/cmd_vel</command_topic>
-        <publish_odom>true</publish_odom>
-        <publish_odom_tf>true</publish_odom_tf>
-        <publish_wheel_tf>true</publish_wheel_tf>
-        <odometry_topic>limo${robot_id}/odom</odometry_topic>
-        <odometry_frame>limo${robot_id}/odom</odometry_frame>
-        <robot_base_frame>limo${robot_id}/base_footprint</robot_base_frame>
-        <odometry_source>1</odometry_source>
-        <ros>
-            <remapping>~/odom:=/odometry</remapping>
-        </ros>
-        </plugin>
+	    <!-- defines limo wheel, laser, depth camera, imu macros-->
+	    <xacro:include filename="$(find limo_description)/urdf/limo.xacro" />
+	    <!-- Variables -->
+	    <xacro:property name="M_PI" value="3.14159"/>
+	    <!-- Vehicle Geometries -->
+	    <xacro:property name="base_x_size" value="0.13" />
+	    <xacro:property name="base_y_size" value="0.12" />
+	    <xacro:property name="base_z_size" value="0.1" />
+	    <xacro:property name="wheelbase" value="0.2"/>
+	    <xacro:property name="track" value="0.13"/>
+	    <xacro:property name="wheel_vertical_offset" value="-0.10" />
+	    <xacro:property name="base_mass" value="2.1557"/>
+	    <xacro:property name="wheel_length" value="0.045" />
+	    <xacro:property name="wheel_radius" value="0.045" />
+	  <link name="limo${robot_id}/base_footprint"/>
+	  <joint name="limo${robot_id}/base_joint" type="fixed">
+	    <parent link="limo${robot_id}/base_footprint"/>
+	    <child link="limo${robot_id}/base_link"/>
+	    <origin xyz="0.0 0.0 0.15" rpy="0 0 0"/>
+	  </joint>
+	    <!-- Base link -->
+	    <link name="limo${robot_id}/base_link">
+		<visual>
+		    <origin xyz="0 0 -0.15" rpy="0 0 1.57" />
+		    <geometry>
+		        <mesh filename="file://$(find limo_description)/meshes/limo_optimal.dae" scale="1 1 1"/>
+		    </geometry>
+		</visual>
+		<collision>
+		    <!--origin xyz="0 0 -0.15" rpy="0 0 1.57" /-->
+		    <origin xyz="0 0 0" rpy="0 0 0" />
+		  <geometry>
+		      <box size="${base_x_size} ${base_y_size} ${base_z_size}"/>
+		  </geometry>
+		</collision>
+	    </link>
+	    <link name="limo${robot_id}/inertial_link">
+		<inertial>
+		    <origin xyz="0.0 0.0 0.0" />
+		    <mass value="${base_mass}" />
+		    <inertia ixx="0.24" ixy="0" ixz="0"
+		             iyy="0.96" iyz="0"
+		             izz="0.96" />
+		</inertial>
+	    </link>
+	    <joint name="limo${robot_id}/inertial_joint" type="fixed">
+		<origin xyz="0 0 0" rpy="0 0 0" />
+		<parent link="limo${robot_id}/base_link" />
+		<child link="limo${robot_id}/inertial_link" />
+	    </joint>
+	    <xacro:limo_laser parent_prefix="limo${robot_id}/base_link" frame_prefix="limo${robot_id}/laser">
+		<origin xyz="0.103 0 -0.034" rpy="0 0 0"/>
+	    </xacro:limo_laser>
+	    <xacro:limo_depth_camera parent_prefix="limo${robot_id}/base_link" frame_prefix="limo${robot_id}/depth_camera">
+		<origin xyz="0.084 0 0.03" rpy="0 0 0"/>
+	    </xacro:limo_depth_camera>
+	    <xacro:limo_imu parent_prefix="limo${robot_id}/base_link" frame_prefix="limo${robot_id}/imu">
+		<origin xyz="0.0 0 -0.1" rpy="0 0 0"/>
+	    </xacro:limo_imu>
+	    <xacro:limo_wheel parent_prefix="limo${robot_id}/base_link" wheel_prefix="limo${robot_id}/front_left" reflect="1">
+		<origin xyz="${wheelbase/2} ${track/2} ${wheel_vertical_offset}" rpy="0 0  0" />
+	    </xacro:limo_wheel>
+	    <xacro:limo_wheel parent_prefix="limo${robot_id}/base_link" wheel_prefix="limo${robot_id}/front_right" reflect="-1">
+		<origin xyz="${wheelbase/2} ${-track/2} ${wheel_vertical_offset}" rpy="${M_PI} 0 0" />
+	    </xacro:limo_wheel>
+	    <xacro:limo_wheel parent_prefix="limo${robot_id}/base_link" wheel_prefix="limo${robot_id}/rear_left" reflect="1">
+		<origin xyz="${-wheelbase/2} ${track/2} ${wheel_vertical_offset}" rpy="0 0 0" />
+	    </xacro:limo_wheel>
+	    <xacro:limo_wheel parent_prefix="limo${robot_id}/base_link" wheel_prefix="limo${robot_id}/rear_right" reflect="-1">
+		<origin xyz="${-wheelbase/2} ${-track/2} ${wheel_vertical_offset}" rpy="${M_PI} 0 0" />
+	    </xacro:limo_wheel>
+	    <xacro:include filename="$(find limo_description)/urdf/limo_transmission.gazebo" />
+	       <!-- Actuator configurations -->
+	    <xacro:limo_wheel_transmission wheel_prefix="limo${robot_id}/front_right" />
+	    <xacro:limo_wheel_transmission wheel_prefix="limo${robot_id}/front_left" />
+	    <xacro:limo_wheel_transmission wheel_prefix="limo${robot_id}/rear_left" />
+	    <xacro:limo_wheel_transmission wheel_prefix="limo${robot_id}/rear_right" />
+        <gazebo>
+	<plugin name="gazebo_ros_control" filename="libgazebo_ros_control.so">
+	    <robotNamespace>/limo$(arg robot_id)</robotNamespace>
+	</plugin>
     </gazebo>
     </xacro:macro>

Commit message: some cleanup

File: limo_description/urdf/limo_four_diff.xacro (robot description, xacro)
@@ -2,5 +2,5 @@
 <robot name="limo" xmlns:xacro="http://ros.org/wiki/xacro">
     <xacro:arg name="robot_id" default="" />
-    <xacro:macro name="limo" params='robot_id'>
+	     <xacro:macro name="limo" params='robot_id'>
 	    <!-- defines limo wheel, laser, depth camera, imu macros-->
 	    <xacro:include filename="$(find limo_description)/urdf/limo.xacro" />
