Commit message: cosmetic changes

File: limo_description/urdf/limo_four_diff.xacro (robot description, xacro)
@@ -1,177 +1,188 @@
 <?xml version="1.0"?>
 <robot name="limo" xmlns:xacro="http://ros.org/wiki/xacro">
-    <xacro:arg name="robot_id" default="" />
-    <xacro:arg name="sensors" default="true" />
-     <xacro:macro name="limo_robot" params='robot_id'>
-	    <!-- defines limo wheel, laser, depth camera, imu macros-->
-    	    <xacro:include filename="$(find limo_description)/urdf/limo.xacro" />
-	    <!-- Variables -->
-	    <xacro:property name="M_PI" value="3.14159"/>
-	    <!-- Vehicle Geometries -->
-	    <xacro:property name="base_x_size" value="0.13" />
-	    <xacro:property name="base_y_size" value="0.12" />
-	    <xacro:property name="base_z_size" value="0.1" />
-	    <xacro:property name="wheelbase" value="0.2"/>
-	    <xacro:property name="track" value="0.13"/>
-	    <xacro:property name="wheel_vertical_offset" value="-0.10" />
-	    <xacro:property name="base_mass" value="2.1557"/>
-	    <xacro:property name="wheel_length" value="0.045" />
-	    <xacro:property name="wheel_radius" value="0.045" />
-	  <!--link name="limo${robot_id}/base_footprint"/-->
-	  <!--joint name="limo${robot_id}/base_joint" type="fixed">
-	    <parent link="limo${robot_id}/base_footprint"/>
-	    <child link="limo${robot_id}/base_link"/>
-	    <origin xyz="0.0 0.0 0.15" rpy="0 0 0"/>
-	  </joint-->
-	    <!-- Base link -->
-	    <link name="limo${robot_id}/base_link">
-		<visual>
-		    <origin xyz="0 0 -0.15" rpy="0 0 1.57" />
-		    <geometry>
-		        <mesh filename="file://$(find limo_description)/meshes/limo_base.dae" scale="1 1 1"/>
-		    </geometry>
-		</visual>
-		<collision>
-		    <!--origin xyz="0 0 -0.15" rpy="0 0 1.57" /-->
-		    <origin xyz="0 0 -0.15" rpy="0 0 1.57" />
-		  <geometry>
-		      <mesh filename="file://$(find limo_description)/meshes/limo_base.dae" scale="1 1 1"/>
-		  </geometry>
-		</collision>
-	    </link>
-	    <link name="limo${robot_id}/inertial_link">
-		<inertial>
-		    <origin xyz="0.0 0.0 0.0" />
-		    <mass value="${base_mass}" />
-		    <inertia ixx="0.24" ixy="0" ixz="0"
-		             iyy="0.96" iyz="0"
-		             izz="0.96" />
-		</inertial>
-	    </link>
-	    <joint name="limo${robot_id}/inertial_joint" type="fixed">
-		<origin xyz="0 0 0" rpy="0 0 0" />
-		<parent link="limo${robot_id}/base_link" />
-		<child link="limo${robot_id}/inertial_link" />
+	<xacro:arg name="robot_id" default="" />
+	<xacro:arg name="sensors" default="true" />
+	<xacro:macro name="limo_robot" params='robot_id'>
+		<!-- defines limo wheel, laser, depth camera, imu macros-->
+		<xacro:include filename="$(find limo_description)/urdf/limo.xacro" />
+		<!-- Variables -->
+		<xacro:property name="M_PI" value="3.14159" />
+		<!-- Vehicle Geometries -->
+		<xacro:property name="base_x_size" value="0.13" />
+		<xacro:property name="base_y_size" value="0.12" />
+		<xacro:property name="base_z_size" value="0.1" />
+		<xacro:property name="wheelbase" value="0.2" />
+		<xacro:property name="track" value="0.13" />
+		<xacro:property name="wheel_vertical_offset" value="-0.10" />
+		<xacro:property name="base_mass" value="2.1557" />
+		<xacro:property name="wheel_length" value="0.045" />
+		<xacro:property name="wheel_radius" value="0.045" />
+		<!-- Base link -->
+		<link name="limo${robot_id}/base_link">
+			<visual>
+				<origin xyz="0 0 -0.15" rpy="0 0 1.57" />
+				<geometry>
+					<mesh filename="file://$(find limo_description)/meshes/limo_base.dae"
+						scale="1 1 1" />
+				</geometry>
+			</visual>
+			<collision>
+				<!--origin
+				xyz="0 0 -0.15" rpy="0 0 1.57" /-->
+				<origin xyz="0 0 -0.15" rpy="0 0 1.57" />
+				<geometry>
+					<mesh filename="file://$(find limo_description)/meshes/limo_base.dae"
+						scale="1 1 1" />
+				</geometry>
+			</collision>
+		</link>
+		<link name="limo${robot_id}/inertial_link">
+			<inertial>
+				<origin xyz="0.0 0.0 0.0" />
+				<mass value="${base_mass}" />
+				<inertia ixx="0.24" ixy="0" ixz="0"
+					iyy="0.96" iyz="0"
+					izz="0.96" />
+			</inertial>
+		</link>
+		<joint name="limo${robot_id}/inertial_joint" type="fixed">
+			<origin xyz="0 0 0" rpy="0 0 0" />
+			<parent link="limo${robot_id}/base_link" />
+			<child link="limo${robot_id}/inertial_link" />
+		</joint>
+		<link name="limo${robot_id}/base_footprint"/>
+			<joint name="limo${robot_id}/base_joint" type="fixed">
+				<parent link="limo${robot_id}/base_link"/>
+				<child link="limo${robot_id}/base_footprint"/>
+			<origin xyz="0.0 0.0 -0.15" rpy="0 0 0"/>
 	    </joint>
-	    <xacro:limo_laser parent_prefix="limo${robot_id}/base_link" frame_prefix="limo${robot_id}/laser">
-		<origin xyz="0.103 0 -0.034" rpy="0 0 0"/>
-	    </xacro:limo_laser>
-	    <xacro:limo_depth_camera parent_prefix="limo${robot_id}/base_link" frame_prefix="limo${robot_id}/depth_camera">
-		<origin xyz="0.084 0 0.03" rpy="0 0 0"/>
-	    </xacro:limo_depth_camera>
-	    <xacro:limo_imu parent_prefix="limo${robot_id}/base_link" frame_prefix="limo${robot_id}/imu">
-		<origin xyz="0.0 0 -0.1" rpy="0 0 0"/>
-	    </xacro:limo_imu>
-	    <xacro:limo_wheel parent_prefix="limo${robot_id}/base_link" wheel_prefix="limo${robot_id}/front_left" reflect="1">
-		<origin xyz="${wheelbase/2} ${track/2} ${wheel_vertical_offset}" rpy="0 0  0" />
-	    </xacro:limo_wheel>
-	    <xacro:limo_wheel parent_prefix="limo${robot_id}/base_link" wheel_prefix="limo${robot_id}/front_right" reflect="-1">
-		<origin xyz="${wheelbase/2} ${-track/2} ${wheel_vertical_offset}" rpy="${M_PI} 0 0" />
-	    </xacro:limo_wheel>
-	    <xacro:limo_wheel parent_prefix="limo${robot_id}/base_link" wheel_prefix="limo${robot_id}/rear_left" reflect="1">
-		<origin xyz="${-wheelbase/2} ${track/2} ${wheel_vertical_offset}" rpy="0 0 0" />
-	    </xacro:limo_wheel>
-	    <xacro:limo_wheel parent_prefix="limo${robot_id}/base_link" wheel_prefix="limo${robot_id}/rear_right" reflect="-1">
-		<origin xyz="${-wheelbase/2} ${-track/2} ${wheel_vertical_offset}" rpy="${M_PI} 0 0" />
-	    </xacro:limo_wheel>
-	    <xacro:include filename="$(find limo_description)/urdf/limo_transmission.gazebo" />
-	       <!-- Actuator configurations -->
-	    <xacro:limo_wheel_transmission wheel_prefix="limo${robot_id}/front_right" />
-	    <xacro:limo_wheel_transmission wheel_prefix="limo${robot_id}/front_left" />
-	    <xacro:limo_wheel_transmission wheel_prefix="limo${robot_id}/rear_left" />
-	    <xacro:limo_wheel_transmission wheel_prefix="limo${robot_id}/rear_right" />
-   <gazebo reference="limo${robot_id}/front_left_wheel_link">
-        <mu1>1.</mu1>
-        <mu2>1.</mu2>
-        <kp>1000000.0</kp>
-        <kd>1.0</kd>
-        <maxVel>1.0</maxVel>
-	<maxContacts>1</maxContacts>
-    </gazebo>
-    <gazebo reference="limo${robot_id}/front_right_wheel_link">
-        <mu1>1.</mu1>
-        <mu2>1.</mu2>
-        <kp>1000000.0</kp>
-        <kd>1.0</kd>
-        <maxVel>1.0</maxVel>
-	<maxContacts>1</maxContacts>
-    </gazebo>
-    <gazebo reference="limo${robot_id}/rear_left_wheel_link">
-        <mu1>0.5</mu1> <!--DIRTY TRICK TO SOLVE ISSUE OF BAD TRACKING DUE TO FRICTION-->
-        <mu2>0.5</mu2>
-        <kp>1000000.0</kp>
-        <kd>1.0</kd>
-        <maxVel>1.0</maxVel>
-	<maxContacts>1</maxContacts>
-    </gazebo>
-    <gazebo reference="limo${robot_id}/rear_right_wheel_link">
-        <mu1>0.5</mu1> <!--DIRTY TRICK TO SOLVE ISSUE OF BAD TRACKING DUE TO FRICTION-->
-        <mu2>0.5</mu2>
-        <kp>1000000.0</kp>
-        <kd>1.0</kd>
-        <maxVel>1.0</maxVel>
-	<maxContacts>1</maxContacts>
-    </gazebo>
-    <!--test with rostopic pub /limo1/cmd_vel geometry_msgs/Twist '{linear: {x: 0.3}, angular: {z: 0.5}}'-->
-	<gazebo>
-		  <disabled_plugin name="diff_drive_controller" filename="libgazebo_ros_diff_drive.so">
-		    <!-- Put all ROS topics inside this namespace -->
-		    <ros>
-		      <nameSpace>limo$(arg robot_id)</nameSpace>
-		    </ros>
-		    <updateRate>50</updateRate>
-		    <leftJoint>limo$(arg robot_id)/front_left_wheel</leftJoint>
-		    <rightJoint>limo$(arg robot_id)/front_right_wheel</rightJoint>
- 		    <!--leftJoint>limo$(arg robot_id)/rear_left_wheel</leftJoint--> <!--DIRTY TRICK TO SOLVE ISSUE OF BAD TRACKING DUE TO FRICTION-->
- 		    <!--rightJoint>limo$(arg robot_id)/rear_right_wheel</rightJoint--> <!--DIRTY TRICK TO SOLVE ISSUE OF BAD TRACKING DUE TO FRICTION-->
-		    <wheelSeparation>0.172</wheelSeparation>
-		    <wheelDiameter>0.095</wheelDiameter>
-		    <!-- Topics are relative to the namespace above -->
-		    <commandTopic>cmd_vel</commandTopic>
-		    <odometryTopic>odom</odometryTopic>
-		    <!-- TF frame IDs must NOT contain '/' -->
-		    <robotBaseFrame>limo$(arg robot_id)/base_link</robotBaseFrame>
-		    <odometryFrame>limo$(arg robot_id)/odom</odometryFrame>
-	            <publishOdom>true</publishOdom>
-		    <odometrySource>1</odometrySource>
-		    <publishWheelJointState>false</publishWheelJointState>
-		    <publishWheelTF>false</publishWheelTF>
-		  </disabled_plugin>
-	        <plugin name="skid_steer_drive_controller" filename="libgazebo_ros_skid_steer_drive.so">
-		    <ros>
-		      <nameSpace>limo$(arg robot_id)</nameSpace>
-		    </ros>
-		    <updateRate>100.0</updateRate>
-		    <leftFrontJoint>limo${robot_id}/front_left_wheel</leftFrontJoint>
-		    <rightFrontJoint>limo${robot_id}/front_right_wheel</rightFrontJoint>
-		    <leftRearJoint>limo${robot_id}/rear_left_wheel</leftRearJoint>
-		    <rightRearJoint>limo${robot_id}/rear_right_wheel</rightRearJoint>
-		    <wheelSeparation>0.164</wheelSeparation>
-		    <wheelDiameter>0.09</wheelDiameter>
-	            <robotBaseFrame>limo${robot_id}/base_link</robotBaseFrame>
-		    <odometryFrame>limo$(arg robot_id)/odom</odometryFrame>
-		    <torque>50</torque>
-		    <!-- Topics are relative to the namespace above -->
-		    <commandTopic>cmd_vel</commandTopic>
-		    <odometryTopic>odom</odometryTopic>
-		    <broadcastTF>true</broadcastTF>
-		       <covariance_x>0.000100</covariance_x>
-            		<covariance_y>0.000100</covariance_y>
-            		<covariance_yaw>0.010000</covariance_yaw>
-		  </plugin>
-		  <!-- Generic publisher for ALL joints in the model -->
-		   <plugin name="joint_state_pub" filename="libgazebo_ros_joint_state_publisher.so">
-		    <ros><namespace>limo$(arg robot_id)</namespace></ros>
-		    <updateRate>100</updateRate>
-                     <alwaysOn>true</alwaysOn>
-	              <jointName>limo$(arg robot_id)/front_left_wheel, limo$(arg robot_id)/rear_left_wheel,limo$(arg robot_id)/front_right_wheel,limo$(arg robot_id)/rear_right_wheel</jointName>
-		  </plugin>
-	</gazebo>
-    <xacro:if value="$(arg sensors)">
-            <xacro:include filename="$(find limo_description)/urdf/limo_sensors.gazebo" />
-      	    <xacro:limo_sensors robot_id="$(arg robot_id)"/>
-      </xacro:if>
-    </xacro:macro>
-    <!-- instantiate the actual robot -->
-    <xacro:limo_robot robot_id="$(arg robot_id)" />
+		<xacro:limo_laser parent_prefix="limo${robot_id}/base_link"
+			frame_prefix="limo${robot_id}/laser">
+			<origin xyz="0.103 0 -0.034" rpy="0 0 0" />
+		</xacro:limo_laser>
+		<xacro:limo_depth_camera parent_prefix="limo${robot_id}/base_link"
+			frame_prefix="limo${robot_id}/depth_camera">
+			<origin xyz="0.084 0 0.03" rpy="0 0 0" />
+		</xacro:limo_depth_camera>
+		<xacro:limo_imu parent_prefix="limo${robot_id}/base_link" frame_prefix="limo${robot_id}/imu">
+			<origin xyz="0.0 0 -0.1" rpy="0 0 0" />
+		</xacro:limo_imu>
+		<xacro:limo_wheel parent_prefix="limo${robot_id}/base_link"
+			wheel_prefix="limo${robot_id}/front_left" reflect="1">
+			<origin xyz="${wheelbase/2} ${track/2} ${wheel_vertical_offset}" rpy="0 0  0" />
+		</xacro:limo_wheel>
+		<xacro:limo_wheel parent_prefix="limo${robot_id}/base_link"
+			wheel_prefix="limo${robot_id}/front_right" reflect="-1">
+			<origin xyz="${wheelbase/2} ${-track/2} ${wheel_vertical_offset}" rpy="${M_PI} 0 0" />
+		</xacro:limo_wheel>
+		<xacro:limo_wheel parent_prefix="limo${robot_id}/base_link"
+			wheel_prefix="limo${robot_id}/rear_left" reflect="1">
+			<origin xyz="${-wheelbase/2} ${track/2} ${wheel_vertical_offset}" rpy="0 0 0" />
+		</xacro:limo_wheel>
+		<xacro:limo_wheel parent_prefix="limo${robot_id}/base_link"
+			wheel_prefix="limo${robot_id}/rear_right" reflect="-1">
+			<origin xyz="${-wheelbase/2} ${-track/2} ${wheel_vertical_offset}" rpy="${M_PI} 0 0" />
+		</xacro:limo_wheel>
+		<xacro:include filename="$(find limo_description)/urdf/limo_transmission.gazebo" />
+		<!-- Actuator configurations -->
+		<xacro:limo_wheel_transmission wheel_prefix="limo${robot_id}/front_right" />
+		<xacro:limo_wheel_transmission wheel_prefix="limo${robot_id}/front_left" />
+		<xacro:limo_wheel_transmission wheel_prefix="limo${robot_id}/rear_left" />
+		<xacro:limo_wheel_transmission wheel_prefix="limo${robot_id}/rear_right" />
+		<gazebo reference="limo${robot_id}/front_left_wheel_link">
+			<mu1>1.</mu1>
+			<mu2>1.</mu2>
+			<kp>1000000.0</kp>
+			<kd>1.0</kd>
+			<maxVel>1.0</maxVel>
+			<maxContacts>1</maxContacts>
+		</gazebo>
+		<gazebo reference="limo${robot_id}/front_right_wheel_link">
+			<mu1>1.</mu1>
+			<mu2>1.</mu2>
+			<kp>1000000.0</kp>
+			<kd>1.0</kd>
+			<maxVel>1.0</maxVel>
+			<maxContacts>1</maxContacts>
+		</gazebo>
+		<gazebo reference="limo${robot_id}/rear_left_wheel_link">
+			<mu1>1.0</mu1>
+			<mu2>1.0</mu2>
+			<kp>1000000.0</kp>
+			<kd>1.0</kd>
+			<maxVel>1.0</maxVel>
+			<maxContacts>1</maxContacts>
+		</gazebo>
+		<gazebo reference="limo${robot_id}/rear_right_wheel_link">
+			<mu1>1.0</mu1>
+			<mu2>1.0</mu2>
+			<kp>1000000.0</kp>
+			<kd>1.0</kd>
+			<maxVel>1.0</maxVel>
+			<maxContacts>1</maxContacts>
+		</gazebo>
+		<gazebo>
+			<disabled_plugin name="diff_drive_controller" filename="libgazebo_ros_diff_drive.so">
+				<!-- Put all ROS topics inside this namespace -->
+				<ros>
+					<nameSpace>limo$(arg robot_id)</nameSpace>
+				</ros>
+				<updateRate>50</updateRate>
+				<leftJoint>limo$(arg robot_id)/front_left_wheel</leftJoint>
+				<rightJoint>limo$(arg robot_id)/front_right_wheel</rightJoint>
+				<wheelSeparation>0.172</wheelSeparation>
+				<wheelDiameter>0.095</wheelDiameter>
+				<!-- Topics are relative to the namespace above -->
+				<commandTopic>cmd_vel</commandTopic>
+				<odometryTopic>odom</odometryTopic>
+				<!-- TF frame IDs must NOT contain '/' -->
+				<robotBaseFrame>limo$(arg robot_id)/base_link</robotBaseFrame>
+				<odometryFrame>limo$(arg robot_id)/odom</odometryFrame>
+				<publishOdom>true</publishOdom>
+				<odometrySource>1</odometrySource>
+				<publishWheelJointState>false</publishWheelJointState>
+				<publishWheelTF>false</publishWheelTF>
+			</disabled_plugin>
+			<plugin name="skid_steer_drive_controller" filename="libgazebo_ros_skid_steer_drive.so">
+				<ros>
+					<nameSpace>limo$(arg robot_id)</nameSpace>
+				</ros>
+				<updateRate>100.0</updateRate>
+				<leftFrontJoint>limo${robot_id}/front_left_wheel</leftFrontJoint>
+				<rightFrontJoint>limo${robot_id}/front_right_wheel</rightFrontJoint>
+				<leftRearJoint>limo${robot_id}/rear_left_wheel</leftRearJoint>
+				<rightRearJoint>limo${robot_id}/rear_right_wheel</rightRearJoint>
+				<wheelSeparation>0.172</wheelSeparation>
+				<wheelDiameter>0.095</wheelDiameter>
+				<!-- Topics are relative to the namespace above -->
+				<commandTopic>cmd_vel</commandTopic>
+				<odometryTopic>odom</odometryTopic>
+				<robotBaseFrame>limo${robot_id}/base_link</robotBaseFrame>
+				<odometryFrame>limo$(arg robot_id)/odom</odometryFrame>
+				<torque>50</torque>
+				<broadcastTF>true</broadcastTF>
+				<covariance_x>0.000100</covariance_x>
+				<covariance_y>0.000100</covariance_y>
+				<covariance_yaw>0.010000</covariance_yaw>
+			</plugin>
+			<!-- Generic publisher for ALL joints in the model -->
+			<plugin name="joint_state_pub" filename="libgazebo_ros_joint_state_publisher.so">
+				<ros>
+					<namespace>limo$(arg robot_id)</namespace>
+				</ros>
+				<updateRate>100</updateRate>
+				<alwaysOn>true</alwaysOn>
+				<jointName>limo$(arg robot_id)/front_left_wheel,
+						   limo$(arg robot_id)/rear_left_wheel,
+						   limo$(arg robot_id)/front_right_wheel,
+						   limo$(arg robot_id)/rear_right_wheel</jointName>
+			</plugin>
+		</gazebo>
+		<xacro:if value="$(arg sensors)">
+			<xacro:include filename="$(find limo_description)/urdf/limo_sensors.gazebo" />
+			<xacro:limo_sensors robot_id="$(arg robot_id)" />
+		</xacro:if>
+	</xacro:macro>
+	<!-- instantiate the actual robot -->
+	<xacro:limo_robot robot_id="$(arg robot_id)" />
 </robot>
